File: clock_PC_and_instruction_reg.sch (EAGLE design)
At the start: 2 parts, among them IC1 74LS245N, IC2 74LS245N

Commit message: Finished all moduled except Logic Control Unit and modified ALU logic
Parts:
- removed IC1, IC2: 74LS245N, 74xx-eu:74LS245N
- added JP1, JP2: (no value), pinhead:PINHD-1X2/90
- added JP3: (no value), pinhead:PINHD-1X1
- added JP4: (no value), pinhead:PINHD-1X8/90
- added U$1: PORT_BOARD, stack_interface:PORT_BOARD
Connections:
- removed net !INPUT_ENABLE: IC1A.G1, IC1A.G2, IC2A.G1, IC2A.G2
- removed net !OE: IC1G$1.!OE
- removed net !OUTPUT_ENABLE: IC1A.G, IC2A.G
- removed net !PC_LOAD: IC1A.LD, IC2A.LD
- removed net !WE: IC1G$1.!WE
- removed net A0: IC1A.B1, IC2A.B1
- removed net A1: IC1A.B2, IC2A.B2
- removed net A10: IC1A.B3, IC2A.B3
- removed net A11: IC1A.B4, IC2A.B4
- removed net A12: IC1A.B5, IC2A.B5
- removed net A13: IC1A.B6, IC2A.B6
- removed net A14: IC1A.B7, IC2A.B7
- removed net A15: IC1A.B8, IC2A.B8
- removed net A2: IC1A.B3, IC2A.B3
- removed net A3: IC1A.B4, IC2A.B4
- removed net A4: IC1A.B5, IC2A.B5
- removed net A5: IC1A.B6, IC2A.B6
- removed net A6: IC1A.B7, IC2A.B7
- removed net A7: IC1A.B8, IC2A.B8
- removed net A8: IC1A.B1, IC2A.B1
- removed net A9: IC1A.B2, IC2A.B2
- removed net ADDR_0: IC1A.D1
- removed net ADDR_1: IC1A.D2
- removed net ADDR_2: IC1A.D3
- removed net ADDR_3: IC1A.D4
- removed net ADDR_4: IC2A.D1
- removed net ADDR_5: IC2A.D2
- removed net ADDR_6: IC2A.D3
- removed net ADDR_7: IC2A.D4
- removed net A_0: IC1A.A, IC2A.A1, IC2A.I0
- removed net A_1: IC1A.B, IC2A.A2, IC2B.I0
- removed net A_10: IC1G$1.A8
- removed net A_11: IC1G$1.A9
- removed net A_12: IC1G$1.A10
- removed net A_13: IC1G$1.A11
- removed net A_14: IC1G$1.A12
- removed net A_15: IC1G$1.A13
- removed net A_2: IC1A.C, IC1G$1.A0, IC2A.A3
- removed net A_3: IC1A.D, IC1G$1.A1, IC2A.A4
- removed net A_4: IC1A.A1, IC1G$1.A2, IC2A.A
- removed net A_5: IC1A.A2, IC1G$1.A3, IC2A.B
- removed net A_6: IC1A.A3, IC1G$1.A4, IC2A.C
- removed net A_7: IC1A.A4, IC1G$1.A5, IC2A.D
- removed net A_8: IC1G$1.A6
- removed net A_9: IC1G$1.A7
- removed net CLOCK: IC1A.CLK, IC2A.CLK
- removed net CLR: IC1A.CLR, IC2A.CLR
- removed net DATA_0: IC1A.D4
- removed net DATA_1: IC1A.D3
- removed net DATA_2: IC1A.D2
- removed net DATA_3: IC1A.D1
- removed net DATA_4: IC2A.D4
- removed net DATA_5: IC2A.D3
- removed net DATA_6: IC2A.D2
- removed net DATA_7: IC2A.D1
- removed net MAR_IN: IC1A.G1, IC1A.G2, IC2A.G1, IC2A.G2
- removed net N$27: IC2A.A2, IC2A.A4, IC2A.O, IC2A.QB
- removed net N$35: IC1A.G, IC1A.Q1, IC2A.G
- removed net N$36: IC1A.Q2
- removed net N$37: IC1A.Q3
- removed net N$38: IC1A.Q4
- removed net N$39: IC2A.Q1
- removed net N$40: IC2A.Q2
- removed net N$41: IC2A.Q3
- removed net N$42: IC2A.Q4
- removed net N$48: IC1A.C4
- removed net PC_ADVANCE: IC1A.CLK
- removed net SUB: IC2A.C0
- removed net UB_0: IC1A.Q4
- removed net UB_1: IC1A.Q3
- removed net UB_2: IC1A.Q2
- removed net UB_3: IC1A.Q1
- removed net UB_4: IC2A.Q4
- removed net UB_5: IC2A.Q3
- removed net UB_6: IC2A.Q2
- removed net UB_7: IC2A.Q1
- new net !II: JP3.1
- new net !PCL: JP1.1
- new net !PCO: JP1.2
- new net HALT: JP2.2
- new net IRO0: JP4.8
- new net IRO7: JP4.1
- new net PC_AD: JP2.1
- net GND: now also U$1.GND; no longer IC1A.D/!U, IC1A.M, IC1A.N, IC1G$1.A14, IC1G$1.GND, IC2A.D/!U, IC2A.M, IC2A.N, IC2G$1.GND
- net N$1: now also U$1.A15; no longer IC1A.C0, IC1A.CTE, IC1G$1.DIS, IC1G$1.DQ0, IC2A.C4, IC2A.CTE
- net N$10: now also U$1.A6; no longer IC2A.B1
- net N$11: now also U$1.A5; no longer IC2A.B2
- net N$12: now also U$1.A4; no longer IC2A.B3
- net N$13: now also U$1.A3; no longer IC2A.B4
- net N$14: now also U$1.A2; no longer IC1A.B1, IC2G$1.CV
- net N$15: now also U$1.A1; no longer IC1A.B2, IC2G$1.TR
- net N$16: now also U$1.A0; no longer IC1A.A1, IC1A.B3
- net N$17: now also U$1.D0; no longer IC1A.A2, IC1A.B4
- net N$18: now also U$1.D1; no longer IC1A.A1, IC1A.A3
- net N$19: now also U$1.D2; no longer IC1A.A2, IC1A.A4
- net N$2: now also U$1.A14; no longer IC1A.QD, IC1G$1.DQ1, IC2A.CLK, IC2A.S4
- net N$20: now also U$1.D3; no longer IC1A.A3, IC1A.A5
- net N$21: now also U$1.D4; no longer IC1A.A4, IC1A.A6
- net N$22: now also U$1.D5; no longer IC1A.A5, IC1A.A7
- net N$23: now also U$1.D6; no longer IC1A.A6, IC1A.A8, IC1A.QA, IC2B.I1
- net N$24: now also U$1.D7; no longer IC1A.A7, IC1A.QB, IC2A.A1, IC2A.I1
- net N$25: now also U$1.CLK; no longer IC1A.A8, IC1A.QC, IC2A.A2
- net N$26: now also U$1.RST; no longer IC2A.A1, IC2A.A3, IC2A.QA
- net N$28: now also JP4.2; no longer IC2A.A3, IC2A.A5, IC2A.QC, IC2B.O
- net N$29: now also JP4.3; no longer IC1G$1.!CE, IC2A.A4, IC2A.A6
- net N$3: now also U$1.A13; no longer IC1A.S1, IC1G$1.DQ2, IC1G$1.THR, IC1G$1.TR, IC2A.QD
- net N$30: now also JP4.4; no longer IC2A.A5, IC2A.A7
- net N$31: now also JP4.5; no longer IC2A.A6, IC2A.A8
- net N$32: now also JP4.6; no longer IC2A.A7
- net N$33: now also JP4.7; no longer IC2A.A8
- net N$4: now also U$1.A12; no longer IC1G$1.DQ3, IC2A.S1, IC2G$1.DIS, IC2G$1.THR
- net N$5: now also U$1.A11; no longer IC1G$1.CV, IC1G$1.DQ4, IC2A.S2
- net N$6: now also U$1.A10; no longer IC1G$1.DQ5, IC1G$1.OUT, IC2A.S3
- net N$7: now also U$1.A9; no longer IC1A.S2, IC1G$1.DQ6
- net N$8: now also U$1.A8; no longer IC1A.S3, IC1G$1.DQ7, IC2G$1.OUT
- net N$9: now also U$1.A7; no longer IC1A.S4
- net VCC: now also U$1.VCC; no longer IC1A.DIR, IC1G$1.!RST, IC1G$1.V+, IC2A.DIR, IC2G$1.!RST, IC2G$1.V+
Other:
- note removed: "加减法器"
- note removed: "按位 AND"

Commit message: Finished all design
Parts:
- removed JP1, JP2: (no value), pinhead:PINHD-1X2/90
- removed JP3: (no value), pinhead:PINHD-1X1
- removed JP4: (no value), pinhead:PINHD-1X8/90
- added IC1: 74LS04N, 74xx-eu:74LS04N
- added JP5: (no value), pinhead:PINHD-1X8/90
- added JP6: (no value), pinhead:PINHD-1X6/90
- added JP7: (no value), pinhead:PINHD-1X15/90
- added JP8: (no value), pinhead:PINHD-1X1
Connections:
- net N$10 renamed I5
- net N$11 renamed I4
- removed net !II: JP3.1
- removed net !PCL: JP1.1
- removed net !PCO: JP1.2
- removed net IRO0: JP4.8
- removed net IRO7: JP4.1
- removed net N$28: JP4.2
- removed net N$29: JP4.3
- removed net N$30: JP4.4
- removed net N$31: JP4.5
- removed net N$32: JP4.6
- removed net N$33: JP4.7
- removed net PC_AD: JP2.1
- new net !INPUT_ENABLE: IC1A.G1, IC1A.G2
- new net ADD: JP5.1
- new net AI: JP7.15
- new net AND: JP5.3
- new net AO: JP7.14
- new net BI: JP7.13
- new net BO: JP7.12
- new net CF: JP5.6, U$1.A11
- new net CI: JP7.11
- new net CLOCK: IC1A.CLK
- new net CLR: IC1A.CLR
- new net CO: JP7.10
- new net D2A_HI_IN: JP6.6
- new net D2A_LO_IN: JP6.5
- new net D2A_OUT: JP6.4
- new net DATA_0: IC1A.D4
- new net DATA_1: IC1A.D3
- new net DATA_2: IC1A.D2
- new net DATA_3: IC1A.D1
- new net DI: JP7.9
- new net DO: JP7.8
- new net EI: JP7.7
- new net EO: JP7.6
- new net HI: JP7.5
- new net HL_TO_ADDR: JP7.1
- new net HO: JP7.4
- new net I2: U$1.A3
- new net I3: U$1.A4
- new net I6: U$1.A7
- new net I7: U$1.A8
- new net INSTRUCTION_IN: U$1.I/O5
- new net LI: JP7.3
- new net LO: JP7.2
- new net MAR_IN: JP6.1, U$1.I/O2
- new net M_READ: JP6.2, U$1.I/O4
- new net M_WRITE: JP6.3, U$1.I/O3
- new net N$10: U$1.A1, U$1.A6
- new net N$11: U$1.A2, U$1.A5
- new net N$27: IC1A.O
- new net NF: JP5.7, U$1.A10
- new net OR: JP5.4
- new net PC_I: U$1.I/O1
- new net PC_O: U$1.I/O0
- new net READY: JP8.1, U$1.A12
- new net RST: IC1A.I
- new net SUB: JP5.2
- new net UB_0: IC1A.Q4
- new net UB_1: IC1A.Q3
- new net UB_2: IC1A.Q2
- new net UB_3: IC1A.Q1
- new net XOR: JP5.5
- new net ZF: JP5.8, U$1.A9
- net GND: now also IC1A.M, IC1A.N, IC1G$1.GND, U$1./CE, U$1./OE
- net HALT: now also U$1.I/O6; no longer JP2.2
- net N$1: now also IC1G$1.DIS, U$1.A0
- net N$2: now also IC1A.O
- net N$26: now also IC1A.I
- net N$3: now also IC1G$1.THR, IC1G$1.TR
- net N$5: now also IC1G$1.CV
- net N$6: now also IC1G$1.OUT
- net VCC: now also IC1G$1.!RST, IC1G$1.V+, U$1./WE
