File: system.sch (EAGLE design)
At the start: 0 parts

Commit message: Added ALU with ADD SUB AND OR and XOR
Other:
- note added: "加减法器"
- note added: "按位 AND"
- note removed: "8位数据总线 8位地址总线 8位指令总线 IO采用在特定地址读写完成"

Commit message: RAM Module halfway done, waiting to add method to manually program the RAM
Parts:
- added IC1, IC2: 74LS245N, 74xx-eu:74LS245N
Connections:
- new net !INPUT_ENABLE: IC1A.G1, IC1A.G2, IC2A.G1, IC2A.G2
- new net !OE: IC1G$1.!OE
- new net !OUTPUT_ENABLE: IC1A.G, IC2A.G
- new net !PC_LOAD: IC1A.LD, IC2A.LD
- new net !WE: IC1G$1.!WE
- new net A0: IC1A.B1, IC2A.B1
- new net A1: IC1A.B2, IC2A.B2
- new net A10: IC1A.B3, IC2A.B3
- new net A11: IC1A.B4, IC2A.B4
- new net A12: IC1A.B5, IC2A.B5
- new net A13: IC1A.B6, IC2A.B6
- new net A14: IC1A.B7, IC2A.B7
- new net A15: IC1A.B8, IC2A.B8
- new net A2: IC1A.B3, IC2A.B3
- new net A3: IC1A.B4, IC2A.B4
- new net A4: IC1A.B5, IC2A.B5
- new net A5: IC1A.B6, IC2A.B6
- new net A6: IC1A.B7, IC2A.B7
- new net A7: IC1A.B8, IC2A.B8
- new net A8: IC1A.B1, IC2A.B1
- new net A9: IC1A.B2, IC2A.B2
- new net ADDR_0: IC1A.D1
- new net ADDR_1: IC1A.D2
- new net ADDR_2: IC1A.D3
- new net ADDR_3: IC1A.D4
- new net ADDR_4: IC2A.D1
- new net ADDR_5: IC2A.D2
- new net ADDR_6: IC2A.D3
- new net ADDR_7: IC2A.D4
- new net A_0: IC1A.A, IC2A.A1, IC2A.I0
- new net A_1: IC1A.B, IC2A.A2, IC2B.I0
- new net A_10: IC1G$1.A8
- new net A_11: IC1G$1.A9
- new net A_12: IC1G$1.A10
- new net A_13: IC1G$1.A11
- new net A_14: IC1G$1.A12
- new net A_15: IC1G$1.A13
- new net A_2: IC1A.C, IC1G$1.A0, IC2A.A3
- new net A_3: IC1A.D, IC1G$1.A1, IC2A.A4
- new net A_4: IC1A.A1, IC1G$1.A2, IC2A.A
- new net A_5: IC1A.A2, IC1G$1.A3, IC2A.B
- new net A_6: IC1A.A3, IC1G$1.A4, IC2A.C
- new net A_7: IC1A.A4, IC1G$1.A5, IC2A.D
- new net A_8: IC1G$1.A6
- new net A_9: IC1G$1.A7
- new net CLOCK: IC1A.CLK, IC2A.CLK
- new net CLR: IC1A.CLR, IC2A.CLR
- new net DATA_0: IC1A.D4
- new net DATA_1: IC1A.D3
- new net DATA_2: IC1A.D2
- new net DATA_3: IC1A.D1
- new net DATA_4: IC2A.D4
- new net DATA_5: IC2A.D3
- new net DATA_6: IC2A.D2
- new net DATA_7: IC2A.D1
- new net GND: IC1A.D/!U, IC1A.M, IC1A.N, IC1G$1.A14, IC1G$1.GND, IC2A.D/!U, IC2A.M, IC2A.N, IC2G$1.GND
- new net MAR_IN: IC1A.G1, IC1A.G2, IC2A.G1, IC2A.G2
- new net N$1: IC1A.C0, IC1A.CTE, IC1G$1.DIS, IC1G$1.DQ0, IC2A.C4, IC2A.CTE
- new net N$10: IC2A.B1
- new net N$11: IC2A.B2
- new net N$12: IC2A.B3
- new net N$13: IC2A.B4
- new net N$14: IC1A.B1, IC2G$1.CV
- new net N$15: IC1A.B2, IC2G$1.TR
- new net N$16: IC1A.A1, IC1A.B3
- new net N$17: IC1A.A2, IC1A.B4
- new net N$18: IC1A.A1, IC1A.A3
- new net N$19: IC1A.A2, IC1A.A4
- new net N$2: IC1A.QD, IC1G$1.DQ1, IC2A.CLK, IC2A.S4
- new net N$20: IC1A.A3, IC1A.A5
- new net N$21: IC1A.A4, IC1A.A6
- new net N$22: IC1A.A5, IC1A.A7
- new net N$23: IC1A.A6, IC1A.A8, IC1A.QA, IC2B.I1
- new net N$24: IC1A.A7, IC1A.QB, IC2A.A1, IC2A.I1
- new net N$25: IC1A.A8, IC1A.QC, IC2A.A2
- new net N$26: IC2A.A1, IC2A.A3, IC2A.QA
- new net N$27: IC2A.A2, IC2A.A4, IC2A.O, IC2A.QB
- new net N$28: IC2A.A3, IC2A.A5, IC2A.QC, IC2B.O
- new net N$29: IC1G$1.!CE, IC2A.A4, IC2A.A6
- new net N$3: IC1A.S1, IC1G$1.DQ2, IC1G$1.THR, IC1G$1.TR, IC2A.QD
- new net N$30: IC2A.A5, IC2A.A7
- new net N$31: IC2A.A6, IC2A.A8
- new net N$32: IC2A.A7
- new net N$33: IC2A.A8
- new net N$35: IC1A.G, IC1A.Q1, IC2A.G
- new net N$36: IC1A.Q2
- new net N$37: IC1A.Q3
- new net N$38: IC1A.Q4
- new net N$39: IC2A.Q1
- new net N$4: IC1G$1.DQ3, IC2A.S1, IC2G$1.DIS, IC2G$1.THR
- new net N$40: IC2A.Q2
- new net N$41: IC2A.Q3
- new net N$42: IC2A.Q4
- new net N$48: IC1A.C4
- new net N$5: IC1G$1.CV, IC1G$1.DQ4, IC2A.S2
- new net N$6: IC1G$1.DQ5, IC1G$1.OUT, IC2A.S3
- new net N$7: IC1A.S2, IC1G$1.DQ6
- new net N$8: IC1A.S3, IC1G$1.DQ7, IC2G$1.OUT
- new net N$9: IC1A.S4
- new net PC_ADVANCE: IC1A.CLK
- new net SUB: IC2A.C0
- new net UB_0: IC1A.Q4
- new net UB_1: IC1A.Q3
- new net UB_2: IC1A.Q2
- new net UB_3: IC1A.Q1
- new net UB_4: IC2A.Q4
- new net UB_5: IC2A.Q3
- new net UB_6: IC2A.Q2
- new net UB_7: IC2A.Q1
- new net VCC: IC1A.DIR, IC1G$1.!RST, IC1G$1.V+, IC2A.DIR, IC2G$1.!RST, IC2G$1.V+

Commit message: Added something about outter bus
Connections:
- new net !HL_TO_ADDR: IC1A.G, IC2A.G
- net GND: now also IC1A.CTE, IC2A.CTE
- net N$1: no longer IC1A.CTE, IC2A.CTE
- net N$35: no longer IC1A.G, IC2A.G

Commit message: Added Regigter A, Register D and ALU module and its PCB
Parts:
- added JP1: (no value), pinhead:PINHD-1X8/90
- added JP2: (no value), pinhead:PINHD-1X2/90
- added U$1: PORT_BOARD, stack_interface:PORT_BOARD
Connections:
- new net CLOCK1: U$1.CLK
- new net N$65: U$1.RST
- new net N$67: JP1.1
- new net N$68: JP1.2
- new net N$69: JP1.3
- new net N$70: JP1.4
- new net N$71: JP1.5
- new net N$72: JP1.6
- new net N$73: JP1.7
- new net N$74: JP1.8
- new net N$75: JP2.2
- new net N$76: JP2.1
- net !OE: now also U$1./OE
- net !WE: now also U$1./WE
- net A_10: now also U$1.A8
- net A_11: now also U$1.A9
- net A_12: now also U$1.A10
- net A_13: now also U$1.A11
- net A_14: now also U$1.A12
- net A_15: now also U$1.A13
- net A_2: now also U$1.A0
- net A_3: now also U$1.A1
- net A_4: now also U$1.A2
- net A_5: now also U$1.A3
- net A_6: now also U$1.A4
- net A_7: now also U$1.A5
- net A_8: now also U$1.A6
- net A_9: now also U$1.A7
- net DATA_0: now also U$1.D0
- net DATA_1: now also U$1.D1
- net DATA_2: now also U$1.D2
- net DATA_3: now also U$1.D3
- net DATA_4: now also U$1.D4
- net DATA_5: now also U$1.D5
- net DATA_6: now also U$1.D6
- net DATA_7: now also U$1.D7
- net GND: now also U$1.A14, U$1.GND
- net N$1: now also U$1.I/O0
- net N$2: now also U$1.I/O1
- net N$29: now also U$1./CE
- net N$3: now also U$1.I/O2
- net N$4: now also U$1.I/O3
- net N$5: now also U$1.I/O4
- net N$6: now also U$1.I/O5
- net N$7: now also U$1.I/O6
- net N$8: now also U$1.I/O7
- net VCC: now also U$1.VCC

Commit message: Finished all moduled except Logic Control Unit and modified ALU logic
Changed lines of the file:
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@@
+</segment>
+</net>
+<net name="N$66" class="0">
+<segment>
+<portref moduleinst="RAM1" port="!WE"/>
+<wire x1="2.54" y1="-5.08" x2="2.54" y2="-7.62" width="0.1524" layer="91"/>
+<wire x1="2.54" y1="-7.62" x2="25.4" y2="-7.62" width="0.1524" layer="91"/>
+<wire x1="25.4" y1="-7.62" x2="25.4" y2="-149.86" width="0.1524" layer="91"/>
+</segment>
+</net>
+<net name="N$77" class="0">
+<segment>
+<wire x1="22.86" y1="-149.86" x2="22.86" y2="-10.16" width="0.1524" layer="91"/>
+<wire x1="22.86" y1="-10.16" x2="0" y2="-10.16" width="0.1524" layer="91"/>
+<portref moduleinst="RAM1" port="!OE"/>
+<wire x1="0" y1="-10.16" x2="0" y2="-5.08" width="0.1524" layer="91"/>
+</segment>
+</net>
+<net name="N$78" class="0">
+<segment>
+<portref moduleinst="ROM1" port="!OE"/>
+<wire x1="-66.04" y1="-35.56" x2="-66.04" y2="-38.1" width="0.1524" layer="91"/>
+<wire x1="-66.04" y1="-38.1" x2="20.32" y2="-38.1" width="0.1524" layer="91"/>
+<wire x1="20.32" y1="-38.1" x2="20.32" y2="-149.86" width="0.1524" layer="91"/>
+</segment>
+</net>
+<net name="N$79" class="0">
+<segment>
+<portref moduleinst="IO_PANEL1" port="EN"/>
+<wire x1="-129.54" y1="-66.04" x2="-129.54" y2="-86.36" width="0.1524" layer="91"/>
+<wire x1="-129.54" y1="-86.36" x2="17.78" y2="-86.36" width="0.1524" layer="91"/>
+<wire x1="17.78" y1="-86.36" x2="17.78" y2="-149.86" width="0.1524" layer="91"/>
+</segment>
+</net>
+<net name="N$80" class="0">
+<segment>
+<portref moduleinst="IO_PANEL1" port="!W!/R"/>
+<wire x1="-132.08" y1="-66.04" x2="-132.08" y2="-88.9" width="0.1524" layer="91"/>
+<wire x1="-132.08" y1="-88.9" x2="15.24" y2="-88.9" width="0.1524" layer="91"/>
+<wire x1="15.24" y1="-88.9" x2="15.24" y2="-149.86" width="0.1524" layer="91"/>
+</segment>
+</net>
+<net name="N$81" class="0">
+<segment>
+<portref moduleinst="IO_PANEL1" port="READY"/>
+<wire x1="-121.92" y1="-66.04" x2="-121.92" y2="-165.1" width="0.1524" layer="91"/>
+<wire x1="-121.92" y1="-165.1" x2="-15.24" y2="-165.1" width="0.1524" layer="91"/>
+</segment>
+</net>
+<net name="N$82" class="0">
+<segment>
+<portref moduleinst="MEMORY_ADDRESS_REGISTOR1" port="MAR_IN"/>
+<wire x1="20.32" y1="121.92" x2="22.86" y2="121.92" width="0.1524" layer="91"/>
+<wire x1="22.86" y1="121.92" x2="22.86" y2="-5.08" width="0.1524" layer="91"/>
+<wire x1="22.86" y1="-5.08" x2="17.78" y2="-5.08" width="0.1524" layer="91"/>
+<wire x1="17.78" y1="-5.08" x2="17.78" y2="-83.82" width="0.1524" layer="91"/>
+<wire x1="17.78" y1="-83.82" x2="12.7" y2="-83.82" width="0.1524" layer="91"/>
+<wire x1="12.7" y1="-149.86" x2="12.7" y2="-83.82" width="0.1524" layer="91"/>
+</segment>
+</net>
+<net name="N$83" class="0">
+<segment>
+<wire x1="40.64" y1="-149.86" x2="40.64" y2="-142.24" width="0.1524" layer="91"/>
+<portref moduleinst="INSTRUCTION_REGISTER1" port="!INPUT_ENABLE"/>
+<wire x1="40.64" y1="-142.24" x2="68.58" y2="-142.24" width="0.1524" layer="91"/>
+<wire x1="68.58" y1="-142.24" x2="68.58" y2="-137.16" width="0.1524" layer="91"/>
+</segment>
+</net>
+<net name="N$84" class="0">
+<segment>
+<portref moduleinst="INSTRUCTION_REGISTER1" port="O0"/>
+<wire x1="45.72" y1="-137.16" x2="45.72" y2="-149.86" width="0.1524" layer="91"/>
+</segment>
+</net>
+<net name="N$85" class="0">
+<segment>
+<portref moduleinst="INSTRUCTION_REGISTER1" port="O1"/>
+<wire x1="48.26" y1="-149.86" x2="48.26" y2="-137.16" width="0.1524" layer="91"/>
+</segment>
+</net>
+<net name="N$86" class="0">
+<segment>
+<portref moduleinst="INSTRUCTION_REGISTER1" port="O2"/>
+<wire x1="50.8" y1="-149.86" x2="50.8" y2="-137.16" width="0.1524" layer="91"/>
+</segment>
+</net>
+<net name="N$87" class="0">
+<segment>
+<portref moduleinst="INSTRUCTION_REGISTER1" port="O3"/>
+<wire x1="53.34" y1="-149.86" x2="53.34" y2="-137.16" width="0.1524" layer="91"/>
+</segment>
+</net>
+<net name="N$88" class="0">
+<segment>
+<portref moduleinst="INSTRUCTION_REGISTER1" port="O4"/>
+<wire x1="55.88" y1="-149.86" x2="55.88" y2="-137.16" width="0.1524" layer="91"/>
+</segment>
+</net>
+<net name="N$89" class="0">
+<segment>
+<portref moduleinst="INSTRUCTION_REGISTER1" port="O5"/>
+<wire x1="58.42" y1="-149.86" x2="58.42" y2="-137.16" width="0.1524" layer="91"/>
+</segment>
+</net>
+<net name="N$90" class="0">
+<segment>
+<portref moduleinst="INSTRUCTION_REGISTER1" port="O6"/>
+<wire x1="60.96" y1="-149.86" x2="60.96" y2="-137.16" width="0.1524" layer="91"/>
+</segment>
+</net>
+<net name="N$91" class="0">
+<segment>
+<portref moduleinst="INSTRUCTION_REGISTER1" port="O7"/>
+<wire x1="63.5" y1="-149.86" x2="63.5" y2="-137.16" width="0.1524" layer="91"/>
+</segment>
+</net>
+<net name="N$92" class="0">
+<segment>
+<wire x1="60.96" y1="-185.42" x2="60.96" y2="-187.96" width="0.1524" layer="91"/>
+<wire x1="60.96" y1="-187.96" x2="137.16" y2="-187.96" width="0.1524" layer="91"/>
+<portref moduleinst="L_REGISTER" port="!OUTPUT_ENABLE"/>
+<wire x1="137.16" y1="-187.96" x2="137.16" y2="-193.04" width="0.1524" layer="91"/>
+</segment>
+</net>
+<net name="N$93" class="0">
+<segment>
+<portref moduleinst="L_REGISTER" port="!INPUT_ENABLE"/>
+<wire x1="134.62" y1="-193.04" x2="134.62" y2="-190.5" width="0.1524" layer="91"/>
+<wire x1="134.62" y1="-190.5" x2="58.42" y2="-190.5" width="0.1524" layer="91"/>
+<wire x1="58.42" y1="-190.5" x2="58.42" y2="-185.42" width="0.1524" layer="91"/>
 </segment>
 </net>

Commit message: Finished all design
Connections:
- removed net !PC_LOAD: IC1A.LD, IC2A.LD
- removed net PC_ADVANCE: IC1A.CLK
- new net CF: U$1.A11
- new net HALT: U$1.I/O6
- new net I2: U$1.A3
- new net I3: U$1.A4
- new net I4: U$1.A5
- new net I5: U$1.A6
- new net I6: U$1.A7
- new net I7: U$1.A8
- new net INSTRUCTION_IN: U$1.I/O5
- new net M_READ: U$1.I/O4
- new net M_WRITE: U$1.I/O3
- new net NF: U$1.A10
- new net PC_I: U$1.I/O1
- new net PC_O: U$1.I/O0
- new net READY: U$1.A12
- new net RST: IC1A.I
- new net ZF: U$1.A9
- net A_0: no longer IC1A.A
- net A_1: no longer IC1A.B
- net A_2: no longer IC1A.C
- net A_3: no longer IC1A.D
- net A_4: no longer IC2A.A
- net A_5: no longer IC2A.B
- net A_6: no longer IC2A.C
- net A_7: no longer IC2A.D
- net GND: now also U$1./CE, U$1./OE; no longer IC1A.CTE, IC1A.D/!U, IC2A.CTE, IC2A.D/!U
- net MAR_IN: now also U$1.I/O2
- net N$1: now also U$1.A0
- net N$10: now also U$1.A1
- net N$11: now also U$1.A2
- net N$2: now also IC1A.O; no longer IC1A.QD, IC2A.CLK
- net N$23: no longer IC1A.QA
- net N$24: no longer IC1A.QB
- net N$25: no longer IC1A.QC
- net N$26: no longer IC2A.QA
- net N$27: no longer IC2A.QB
- net N$28: no longer IC2A.QC
- net N$3: no longer IC2A.QD
- net VCC: now also U$1./WE
